Commit message: Add lidar to scout-mini simulation model

File: scout/scout_description/urdf/mini.xacro (robot description, xacro)
@@ -97,3 +97,29 @@
     <!-- Gazebo definitions  -->
     <xacro:include filename="$(find scout_description)/urdf/scout_mini.gazebo" />
+    <joint name="hokuyo_joint" type="fixed">
+        <axis xyz="0 1 0" />
+        <origin xyz="0 0 0.088" rpy="0 0 0"/>
+        <parent link="base_link"/>
+        <child link="hokuyo_link"/>
+    </joint>
+    <!-- Hokuyo Laser -->
+    <link name="hokuyo_link">
+        <collision>
+        <origin xyz="0 0 0" rpy="0 0 0"/>
+        <geometry>
+        <box size="0.1 0.1 0.1"/>
+        </geometry>
+        </collision>
+        <visual>
+        <origin xyz="0 0 0" rpy="0 0 0"/>
+        <geometry>
+            <mesh filename="package://scout_description/meshes/hokuyo.dae"/>
+        </geometry>
+        </visual>
+        <inertial>
+        <mass value="1e-5" />
+        <origin xyz="0 0 0" rpy="0 0 0"/>
+        <inertia ixx="1e-6" ixy="0" ixz="0" iyy="1e-6" iyz="0" izz="1e-6" />
+        </inertial>
+    </link>
 </robot>

Commit message: Edit lidar attach point, add realsense camera

File: scout/scout_description/urdf/mini.xacro (robot description, xacro)
@@ -99,5 +99,5 @@
     <joint name="hokuyo_joint" type="fixed">
         <axis xyz="0 1 0" />
-        <origin xyz="0 0 0.088" rpy="0 0 0"/>
+        <origin xyz="0 0 0.14" rpy="0 0 0"/>
         <parent link="base_link"/>
         <child link="hokuyo_link"/>
@@ -123,3 +123,7 @@
         </inertial>
     </link>
+    <xacro:include filename="$(find scout_description)/urdf/_d435.urdf.xacro" />
+    <xacro:sensor_d435 parent="base_link">
+        <origin xyz="0.1 0 0.1" rpy="0 0 0"/>
+    </xacro:sensor_d435>
 </robot>

Commit message: Include lidar data in scout_mini.gazebo into mini.xacro

File: scout/scout_description/urdf/mini.xacro (robot description, xacro)
@@ -123,7 +123,91 @@
         </inertial>
     </link>
+    <gazebo reference="hokuyo_link">
+        <sensor type="ray" name="head_hokuyo_sensor">
+        <pose>0 0 0 0 0 0</pose>
+        <visualize>true</visualize>
+        <update_rate>40</update_rate>
+        <ray>
+            <scan>
+            <horizontal>
+                <samples>720</samples>
+                <resolution>1</resolution>
+                <min_angle>-1.570796</min_angle>
+                <max_angle>1.570796</max_angle>
+            </horizontal>
+            </scan>
+            <range>
+            <min>0.10</min>
+            <max>5.0</max>
+            <resolution>0.01</resolution>
+            </range>
+            <noise>
+            <type>gaussian</type>
+            <!-- Noise parameters based on published spec for Hokuyo laser
+                achieving "+-30mm" accuracy at range < 10m.  A mean of 0.0m and
+                stddev of 0.01m will put 99.7% of samples within 0.03m of the true
+                reading. -->
+            <mean>0.0</mean>
+            <stddev>0.01</stddev>
+            </noise>
+        </ray>
+        <plugin name="gazebo_ros_head_hokuyo_controller" filename="libgazebo_ros_laser.so">
+            <topicName>/scout/laser/scan</topicName>
+            <frameName>hokuyo_link</frameName>
+        </plugin>
+        </sensor>
+    </gazebo>
+    <!-- realsense camera -->
+    <!-- Refer ugv_gazebo_sim/scout/scout_description/_d435.gazebo.xacro -->
+    <!-- Refer ugv_gazebo_sim/scout/scout_description/_d435.urdf.xacro -->
     <xacro:include filename="$(find scout_description)/urdf/_d435.urdf.xacro" />
     <xacro:sensor_d435 parent="base_link">
         <origin xyz="0.1 0 0.1" rpy="0 0 0"/>
     </xacro:sensor_d435>
+    <!-- IMU sensor -->
+    <joint name="imu_joint" type="fixed">
+        <axis xyz="1 0 0"/> <!-- 0 1 0 -->
+        <origin xyz="0 0 0.1"/>
+        <parent link="base_link"/>
+        <child link="imu_link"/>
+    </joint>
+    <link name="imu_link">
+        <inertial>
+            <mass value="0.001"/>
+            <origin rpy="0 0 0" xyz="0 0 0"/>
+            <inertia ixx="0.0001" ixy="0" ixz="0" iyy="0.000001" iyz="0" izz="0.0001"/>
+        </inertial>
+        <visual>
+            <origin rpy="0 0 0" xyz="0 0 0"/>
+            <geometry>
+                <box size="0.001 0.001 0.001"/>
+            </geometry>
+        </visual>
+        <collision>
+            <origin rpy="0 0 0" xyz="0 0 0"/>
+            <geometry>
+                <box size=".001 .001 .001"/>
+            </geometry>
+        </collision>
+    </link>
+    <gazebo reference="imu_link">
+        <gravity>true</gravity>
+        <sensor name="imu_sensor" type="imu">
+            <always_on>true</always_on>
+            <update_rate>50</update_rate>
+            <visualize>true</visualize>
+            <topic>__default_topic__</topic>
+            <plugin filename="libgazebo_ros_imu_sensor.so" name="imu_plugin">
+                <topicName>imu</topicName>
+                <bodyName>imu_link</bodyName>
+                <updateRateHZ>10.0</updateRateHZ>
+                <gaussianNoise>2.89e-08</gaussianNoise>
+                <xyzOffset>0 0 0</xyzOffset>
+                <rpyOffset>0 0 0</rpyOffset>
+                <frameName>imu_link</frameName>
+                <initialOrientationAsReference>false</initialOrientationAsReference>
+            </plugin>
+            <pose>0 0 0 0 0 0</pose>
+        </sensor>
+    </gazebo>
 </robot>

Commit message: Edit  scout_skid_steer, Add base_footprint

File: scout/scout_description/urdf/mini.xacro (robot description, xacro)
@@ -42,4 +42,10 @@
         </collision>
     </link>
+     <link name="base_footprint"/>
+     <joint name="base_footprint_joint" type="fixed">
+        <origin xyz="0 0 ${wheel_vertical_offset - wheel_radius / 2}" rpy="0 0 0" />
+        <parent link="base_link" />
+        <child link="base_footprint" />
+    </joint>
     <!-- <joint name="chassis_link_joint" type="fixed">
         <origin xyz="0 0 ${wheel_radius - wheel_vertical_offset}" rpy="0 0 0" />

Commit message: Add Odometry

File: scout/scout_description/urdf/mini.xacro (robot description, xacro)
@@ -22,4 +22,12 @@
     <xacro:property name="wheel_length" value="0.8e-01" />
     <xacro:property name="wheel_radius" value="1.600e-01" />
+    <link name="base_footprint">
+        <origin xyz="0 0 0" rpy="0 0 0" />
+    </link>
+     <joint name="base_footprint_joint" type="fixed">
+        <origin xyz="0 0 ${-wheel_vertical_offset + wheel_radius / 2}" rpy="0 0 0" />
+        <parent link="base_footprint" />
+        <child link="base_link" />
+    </joint>
     <!-- Base link -->
     <link name="base_link">
@@ -42,10 +50,4 @@
         </collision>
     </link>
-     <link name="base_footprint"/>
-     <joint name="base_footprint_joint" type="fixed">
-        <origin xyz="0 0 ${wheel_vertical_offset - wheel_radius / 2}" rpy="0 0 0" />
-        <parent link="base_link" />
-        <child link="base_footprint" />
-    </joint>
     <!-- <joint name="chassis_link_joint" type="fixed">
         <origin xyz="0 0 ${wheel_radius - wheel_vertical_offset}" rpy="0 0 0" />
@@ -221,6 +223,6 @@
             <alwaysOn>true</alwaysOn>
             <updateRate>50.0</updateRate>
-            <bodyName>base_link</bodyName>
-            <topicName>odom</topicName>
+            <bodyName>base_footprint</bodyName>
+            <topicName>gt_odom</topicName>
             <gaussianNoise>0.01</gaussianNoise>
             <frameName>map</frameName>

Commit message: Edit scout simulator setting

File: scout/scout_description/urdf/mini.xacro (robot description, xacro)
@@ -176,5 +176,5 @@
     <joint name="imu_joint" type="fixed">
         <axis xyz="1 0 0"/> <!-- 0 1 0 -->
-        <origin xyz="0 0 0.1"/>
+        <origin xyz="-0.05 0 0.14"/>
         <parent link="base_link"/>
         <child link="imu_link"/>

File: scout/scout_description/urdf/scout_mini_wheel_1.xacro (robot description, xacro)
@@ -59,4 +59,12 @@
                   filename="package://scout_description/meshes/wheel.dae" />
               </geometry>
+              <surface>
+                <friction>
+                  <ode>
+                    <mu>1.0</mu>
+                    <mu2>1.0</mu2>
+                  </ode>
+                </friction>
+              </surface>
             </collision>
         </link>

File: scout/scout_description/urdf/scout_mini_wheel_2.xacro (robot description, xacro)
@@ -59,4 +59,12 @@
                   filename="package://scout_description/meshes/wheel.dae" />
               </geometry>
+              <surface>
+                <friction>
+                  <ode>
+                    <mu>1.0</mu>
+                    <mu2>1.0</mu2>
+                  </ode>
+                </friction>
+              </surface>
             </collision>
         </link>

File: scout/scout_description/urdf/scout_mini_wheel_3.xacro (robot description, xacro)
@@ -59,4 +59,12 @@
                   filename="package://scout_description/meshes/wheel.dae" />
               </geometry>
+              <surface>
+                <friction>
+                  <ode>
+                    <mu>1.0</mu>
+                    <mu2>1.0</mu2>
+                  </ode>
+                </friction>
+              </surface>
             </collision>
         </link>

File: scout/scout_description/urdf/scout_mini_wheel_4.xacro (robot description, xacro)
@@ -59,4 +59,12 @@
                   filename="package://scout_description/meshes/wheel.dae" />
               </geometry>
+              <surface>
+                <friction>
+                  <ode>
+                    <mu>1.0</mu>
+                    <mu2>1.0</mu2>
+                  </ode>
+                </friction>
+              </surface>
             </collision>
         </link>

Commit message: Tested ros navigation stack

File: scout/scout_description/urdf/mini.xacro (robot description, xacro)
@@ -35,5 +35,5 @@
             <origin
                     xyz="0 0 0.0"
-                    rpy="1.57 0 1.57" />
+                    rpy="1.57 0 -1.57" />
             <geometry>
                 <mesh filename="package://scout_description/meshes/scout_mini_base_link2.dae" />
@@ -43,8 +43,7 @@
             <origin
                     xyz="0 0 0"
-                    rpy="1.57 0 1.57" />
+                    rpy="1.57 0 -1.57" />
           <geometry>
-            <mesh
-              filename="package://scout_description/meshes/scout_mini_base_link2.dae" />
+            <mesh filename="package://scout_description/meshes/scout_mini_base_link2.dae" />
           </geometry>
         </collision>
@@ -230,5 +229,5 @@
             <bodyName>base_footprint</bodyName>
             <topicName>odom_groundtruth</topicName>
-            <gaussianNoise>0.01</gaussianNoise>
+            <gaussianNoise>0.0</gaussianNoise>
             <frameName>world</frameName>
             <xyzOffsets>0 0 0</xyzOffsets>

Commit message: Fix wheel radius

File: scout/scout_description/urdf/mini.xacro (robot description, xacro)
@@ -21,5 +21,7 @@
     <xacro:property name="wheel_vertical_offset" value="-0.160000047342231" />-->
     <xacro:property name="wheel_length" value="0.8e-01" />
-    <xacro:property name="wheel_radius" value="1.600e-01" />
+    <!-- <xacro:property name="wheel_radius" value="1.600e-01" /> -->
+    <!-- SCOUT mini wheel radius is 0.8e-01 -->
+    <xacro:property name="wheel_radius" value="0.8e-01" />
     <!-- Base link -->
     <link name="base_link">

Commit message: Add sensors to mini.xacro

File: scout/scout_description/urdf/mini.xacro (robot description, xacro)
@@ -1,7 +1,38 @@
 <?xml version="1.0"?>
-<robot name="scout_mini"
-    xmlns:xacro="http://ros.org/wiki/xacro">
+<robot name="scout_mini" xmlns:xacro="http://ros.org/wiki/xacro">
     <xacro:arg name="robot_namespace" default="/" />
     <xacro:arg name="urdf_extras" default="empty.urdf" />
+    <!-- Sensors Configuration -->
+    <xacro:arg name="2d_lidar" default="true" />
+    <xacro:arg name="3d_lidar" default="false" />
+    <xacro:arg name="camera" default="true" />
+    <xacro:arg name="visualize" default="true" />
+    <!-- GPU setting -->
+    <xacro:arg name="gpu" default="true" />
+    <xacro:property name="gpu" value="$(arg gpu)" />
+    <!-- Lidar Common parameters -->
+    <xacro:property name="lidar_pose" default="0 0 0.14" />
+    <xacro:property name="lidar_orientation" default="0 0 0" />
+    <!-- 2D Lidar parameters -->
+    <xacro:arg name="2d_lidar_topic" default="/hokuyo/scan" />
+    <!-- 3D Lidar parameters -->
+    <!-- 3d_lidar : VLP-16, HDL32E -->
+    <xacro:arg name="3d_lidar_name" default="VLP-16" />
+    <!-- <xacro:arg name="3d_lidar_name" default="HDL-32E" />  -->
+    <!-- Camera Common parameters -->
+    <xacro:arg name="camera_pose" default="0.13 0 0.1" />
+    <xacro:arg name="camera_orientation" default="0 0 0" />
+    <!-- Camera : rgb, openni-kinect, realsense-d435 -->
+    <!-- <xacro:arg name="camera_name" default="rgb" /> -->
+    <!-- <xacro:arg name="camera_name" default="openni-kinect" /> -->
+    <xacro:arg name="camera_name" default="realsense-d435" />
+    <!-- Realsense Camera parameters -->
+    <xacro:arg name="camera_pointcloud" default="true" />
+    <!-- IMU parameters -->
+    <xacro:arg name="imu" default="true" />
+    <xacro:arg name="imu_topic" default="/imu" />
+    <xacro:arg name="imu_pose" default="0 0 0.07" />
+    <xacro:arg name="imu_orientation" default="0 0 0" />
+    <!-- SCOUT mini wheel 3D file -->
     <xacro:include filename="$(find scout_description)/urdf/scout_mini_wheel_1.xacro" />
     <xacro:include filename="$(find scout_description)/urdf/scout_mini_wheel_2.xacro" />
@@ -17,7 +48,4 @@
     <xacro:property name="track" value="0.416503"/>
     <xacro:property name="wheel_vertical_offset" value="-0.100998" />
-<!--    <xacro:property name="track" value="0.3426" />
-    <xacro:property name="wheelbase" value="0.3181"/>
-    <xacro:property name="wheel_vertical_offset" value="-0.160000047342231" />-->
     <xacro:property name="wheel_length" value="0.8e-01" />
     <!-- <xacro:property name="wheel_radius" value="1.600e-01" /> -->
@@ -35,11 +63,8 @@
         </visual>
         <collision>
-            <origin
-                    xyz="0 0 0"
-                    rpy="1.57 0 -1.57" />
-          <geometry>
-            <mesh
-              filename="package://scout_description/meshes/scout_mini_base_link2.dae" />
-          </geometry>
+            <origin xyz="0 0 0" rpy="1.57 0 -1.57" />
+            <geometry>
+                <mesh filename="package://scout_description/meshes/scout_mini_base_link2.dae" />
+            </geometry>
         </collision>
     </link>
@@ -111,3 +136,32 @@
         </plugin>
     </gazebo>
+    <!-- SENSORS -->
+    <!-- SENSORS -->
+    <!-- SENSORS -->
+    <!-- SENSORS -->
+    <!-- SENSORS -->
+    <!-- 2D hokuyo lidar -->
+    <xacro:if value="$(arg 2d_lidar)" >
+        <xacro:include filename="$(find scout_description)/urdf/hokuyo_2d.xacro" />
+        <xacro:hokuyo_lidar parent_link="base_link" topicName="$(arg 2d_lidar_topic)" visualize="$(arg visualize)" gpu="${gpu}">
+            <origin xyz="${lidar_pose}" rpy="${lidar_orientation}" />
+        </xacro:hokuyo_lidar>
+    </xacro:if>
+    <!-- 3D Velodyne lidar -->
+    <xacro:if value="$(arg 3d_lidar)" >
+        <xacro:include filename="$(find scout_description)/urdf/$(arg 3d_lidar_name).xacro" />
+        <xacro:scout_3d_lidar parent_link="base_link" visualize="$(arg visualize)" gpu="${gpu}" xyz="${lidar_pose}" rpy="${lidar_orientation}" />
+    </xacro:if>
+    <!-- Camera -->
+    <xacro:if value="$(arg camera)" >
+        <xacro:include filename="$(find scout_description)/urdf/$(arg camera_name).xacro" />
+        <xacro:scout_camera parent_link="base_link" name="camera" topics_ns="camera" publish_pointcloud="$(arg camera_pointcloud)" visualize="$(arg visualize)" xyz="$(arg camera_pose)" rpy="$(arg camera_orientation)" />
+    </xacro:if>
+    <!-- IMU -->
+    <xacro:if value="$(arg imu)" >
+        <xacro:include filename="$(find scout_description)/urdf/imu.xacro" />
+        <xacro:IMU parent_link="base_link" topicName="$(arg imu_topic)">
+            <origin xyz="$(arg imu_pose)" rpy="$(arg imu_orientation)" />
+        </xacro:IMU>
+    </xacro:if>
 </robot>
