Commit message: Add gps, edit sensor xacro files

File: scout/scout_description/urdf/hokuyo_2d.xacro (robot description, xacro)
@@ -6,5 +6,5 @@
         <xacro:property name="samples" default="720" />
         <xacro:property name="min_range" default="0.10" />
-        <xacro:property name="max_range" default="5.0" />
+        <xacro:property name="max_range" default="15.0" />
         <xacro:property name="min_angle" default="-3.1415" />
         <xacro:property name="max_angle" default="3.1415" />

File: scout/scout_description/urdf/mini.xacro (robot description, xacro)
@@ -7,6 +7,8 @@
     <xacro:arg name="3d_lidar" default="false" />
     <xacro:arg name="camera" default="true" />
-    <xacro:arg name="visualize" default="true" />
-    <!-- GPU setting -->
+    <xacro:arg name="imu" default="true" />
+    <xacro:arg name="gps" default="false" />
+    <xacro:arg name="visualize" default="false" />
+    <!-- GPU setting for Lidar processing -->
     <xacro:arg name="gpu" default="true" />
     <xacro:property name="gpu" value="$(arg gpu)" />
@@ -25,13 +27,16 @@
     <!-- Camera : rgb, openni-kinect, realsense-d435 -->
     <!-- <xacro:arg name="camera_name" default="rgb" /> -->
-    <xacro:arg name="camera_name" default="openni-kinect" />
-    <!-- <xacro:arg name="camera_name" default="realsense-d435" /> -->
+    <!-- <xacro:arg name="camera_name" default="openni-kinect" /> -->
+    <xacro:arg name="camera_name" default="realsense-d435" />
     <!-- Realsense Camera parameters -->
     <xacro:arg name="camera_pointcloud" default="true" />
     <!-- IMU parameters -->
-    <xacro:arg name="imu" default="true" />
     <xacro:arg name="imu_topic" default="/imu" />
     <xacro:arg name="imu_pose" default="0 0 0.07" />
     <xacro:arg name="imu_orientation" default="0 0 0" />
+    <!-- GPS parameters -->
+    <xacro:arg name="gps_topic" default="/gps" />
+    <xacro:arg name="gps_pose" default="-0.2 0 0.07" />
+    <xacro:arg name="gps_orientation" default="0 0 0" />
     <!-- SCOUT mini wheel 3D file -->
     <xacro:include filename="$(find scout_description)/urdf/scout_mini_wheel_1.xacro" />
@@ -52,4 +57,12 @@
     <!-- SCOUT mini wheel radius is 0.8e-01 -->
     <xacro:property name="wheel_radius" value="0.8e-01" />
+    <link name="base_footprint">
+        <origin xyz="0 0 0" rpy="0 0 0" />
+    </link>
+     <joint name="base_footprint_joint" type="fixed">
+        <origin xyz="0 0 ${-wheel_vertical_offset + wheel_radius}" rpy="0 0 0" />
+        <parent link="base_footprint" />
+        <child link="base_link" />
+    </joint>
     <!-- Base link -->
     <link name="base_link">
@@ -131,5 +144,5 @@
             <topicName>odom_gazebo</topicName>
             <gaussianNoise>0.0</gaussianNoise>
-            <frameName>world</frameName>
+            <frameName>map</frameName>
             <xyzOffsets>0 0 0</xyzOffsets>
             <rpyOffsets>0 0 0</rpyOffsets>
@@ -165,3 +178,10 @@
         </xacro:IMU>
     </xacro:if>
+    <!-- GPS -->
+    <xacro:if value="$(arg gps)" >
+        <xacro:include filename="$(find scout_description)/urdf/gps.xacro" />
+        <xacro:GPS parent_link="base_link" topicName="$(arg gps_topic)">
+            <origin xyz="$(arg gps_pose)" rpy="$(arg gps_orientation)" />
+        </xacro:GPS>
+    </xacro:if>
 </robot>

File: scout/scout_description/urdf/openni-kinect.xacro (robot description, xacro)
@@ -15,5 +15,5 @@
                 <origin xyz="0 0 0" rpy="0 0 0"/>
                 <geometry>
-                    <box size="0.05 0.05 0.05"/>
+                    <box size="0.02 0.05 0.02"/>
                 </geometry>
             </collision>

File: scout/scout_description/urdf/rgb.xacro (robot description, xacro)
@@ -15,5 +15,5 @@
                 <origin xyz="0 0 0" rpy="0 0 0"/>
                 <geometry>
-                    <box size="0.05 0.05 0.05"/>
+                    <box size="0.02 0.05 0.02"/>
                 </geometry>
             </collision>
