Commit message: Edit xacro files and launch file for passing sensor arguments

File: scout/scout_description/urdf/gps.xacro (robot description, xacro)
@@ -3,5 +3,6 @@
 <!-- https://classic.gazebosim.org/tutorials?tut=ros_gzplugins#Camera -->
 <robot xmlns:xacro="http://ros.org/wiki/xacro" name="scout_camera">
-    <xacro:macro name="GPS" params="parent_link topicName *joint_pose">
+    <xacro:macro name="GPS" params="parent_link *joint_pose">
+        <xacro:property name="topicName"    default="/gps" />
         <joint name="gps_joint" type="fixed">
             <axis xyz="0 1 0" />

File: scout/scout_description/urdf/hokuyo_2d.xacro (robot description, xacro)
@@ -3,10 +3,11 @@
 <!-- https://classic.gazebosim.org/tutorials?tut=ros_gzplugins#GPULaser -->
 <robot xmlns:xacro="http://ros.org/wiki/xacro" name="scout_lidar">
-    <xacro:macro name="hokuyo_lidar" params="parent_link topicName visualize:=false *joint_pose gpu:=false">
-        <xacro:property name="samples" default="720" />
-        <xacro:property name="min_range" default="0.10" />
-        <xacro:property name="max_range" default="15.0" />
-        <xacro:property name="min_angle" default="-3.1415" />
-        <xacro:property name="max_angle" default="3.1415" />
+    <xacro:macro name="hokuyo_lidar" params="parent_link visualize:=false *joint_pose gpu:=false">
+        <xacro:property name="topicName"    default="/hokuyo/scan" />
+        <xacro:property name="samples"      default="720"          />
+        <xacro:property name="min_range"    default="0.10"         />
+        <xacro:property name="max_range"    default="15.0"         />
+        <xacro:property name="min_angle"    default="-3.1415"      />
+        <xacro:property name="max_angle"    default="3.1415"       />
         <link name="hokuyo_link">
             <collision>

File: scout/scout_description/urdf/imu.xacro (robot description, xacro)
@@ -3,5 +3,6 @@
 <!-- https://classic.gazebosim.org/tutorials?tut=ros_gzplugins#GPULaser -->
 <robot xmlns:xacro="http://ros.org/wiki/xacro" name="scout_imu">
-    <xacro:macro name="IMU" params="parent_link topicName *joint_pose">
+    <xacro:macro name="IMU" params="parent_link *joint_pose">
+        <xacro:property name="topicName"    default="/imu" />
         <link name="imu_link">
             <inertial>

File: scout/scout_description/urdf/mini.xacro (robot description, xacro)
@@ -4,39 +4,59 @@
     <xacro:arg name="urdf_extras" default="empty.urdf" />
     <!-- Sensors Configuration -->
-    <xacro:arg name="2d_lidar" default="true" />
-    <xacro:arg name="3d_lidar" default="false" />
-    <xacro:arg name="camera" default="true" />
-    <xacro:arg name="imu" default="true" />
-    <xacro:arg name="gps" default="false" />
-    <xacro:arg name="visualize" default="false" />
+    <xacro:arg name="hokuyo_lidar"  default="true"      />
+    <xacro:arg name="velodyne_lidar"  default="false"     />
+    <xacro:arg name="camera"    default="true"      />
+    <xacro:arg name="imu"       default="true"      />
+    <xacro:arg name="gps"       default="true"      />
+    <xacro:arg name="visualize" default="false"     />
     <!-- GPU setting for Lidar processing -->
-    <xacro:arg name="gpu" default="true" />
-    <xacro:property name="gpu" value="$(arg gpu)" />
+    <xacro:arg name="gpu"       default="true"      />
+    <xacro:property name="gpu"  value="$(arg gpu)"  />
     <!-- Lidar Common parameters -->
-    <xacro:property name="lidar_pose" default="0 0 0.14" />
-    <xacro:property name="lidar_orientation" default="0 0 0" />
-    <!-- 2D Lidar parameters -->
-    <xacro:arg name="2d_lidar_topic" default="/hokuyo/scan" />
+    <xacro:arg name="lidar_x"       default="0"     />
+    <xacro:arg name="lidar_y"       default="0"     />
+    <xacro:arg name="lidar_z"       default="0.14"  />
+    <xacro:arg name="lidar_roll"    default="0"     />
+    <xacro:arg name="lidar_pitch"   default="0"     />
+    <xacro:arg name="lidar_yaw"     default="0"     />
+    <xacro:property name="lidar_pose" default="$(arg lidar_x) $(arg lidar_y) $(arg lidar_z)" />
+    <xacro:property name="lidar_orientation" default="$(arg lidar_roll) $(arg lidar_pitch) $(arg lidar_yaw)" />
     <!-- 3D Lidar parameters -->
     <!-- 3d_lidar : VLP-16, HDL32E -->
-    <xacro:arg name="3d_lidar_name" default="VLP-16" />
-    <!-- <xacro:arg name="3d_lidar_name" default="HDL-32E" />  -->
+    <xacro:arg name="velodyne_lidar_name" default="VLP-16" />
+    <!-- <xacro:arg name="velodyne_lidar_name" default="HDL-32E" />  -->
     <!-- Camera Common parameters -->
-    <xacro:arg name="camera_pose" default="0.13 0 0.1" />
-    <xacro:arg name="camera_orientation" default="0 0 0" />
+    <xacro:arg name="camera_x"       default="0.13" />
+    <xacro:arg name="camera_y"       default="0"    />
+    <xacro:arg name="camera_z"       default="0.1"  />
+    <xacro:arg name="camera_roll"    default="0"    />
+    <xacro:arg name="camera_pitch"   default="0"    />
+    <xacro:arg name="camera_yaw"     default="0"    />
+    <xacro:property name="camera_pose" default="$(arg camera_x) $(arg camera_y) $(arg camera_z) " />
+    <xacro:property name="camera_orientation" default="$(arg camera_roll) $(arg camera_pitch) $(arg camera_yaw) " />
     <!-- Camera : rgb, openni-kinect, realsense-d435 -->
     <!-- <xacro:arg name="camera_name" default="rgb" /> -->
     <!-- <xacro:arg name="camera_name" default="openni-kinect" /> -->
     <xacro:arg name="camera_name" default="realsense-d435" />
-    <!-- Realsense Camera parameters -->
+    <!-- openni-kinct, realsense parameters -->
     <xacro:arg name="camera_pointcloud" default="true" />
     <!-- IMU parameters -->
-    <xacro:arg name="imu_topic" default="/imu" />
-    <xacro:arg name="imu_pose" default="0 0 0.07" />
-    <xacro:arg name="imu_orientation" default="0 0 0" />
+    <xacro:arg name="imu_x"               default="-0.1"  />
+    <xacro:arg name="imu_y"               default="0"     />
+    <xacro:arg name="imu_z"               default="0.07"  />
+    <xacro:arg name="imu_roll"            default="0"     />
+    <xacro:arg name="imu_pitch"           default="0"     />
+    <xacro:arg name="imu_yaw"             default="0"     />
+    <xacro:property name="imu_pose" default="$(arg imu_x) $(arg imu_y) $(arg imu_z)" />
+    <xacro:property name="imu_orientation" default="$(arg imu_roll) $(arg imu_pitch) $(arg imu_yaw) " />
     <!-- GPS parameters -->
-    <xacro:arg name="gps_topic" default="/gps" />
-    <xacro:arg name="gps_pose" default="-0.2 0 0.07" />
-    <xacro:arg name="gps_orientation" default="0 0 0" />
+    <xacro:arg name="gps_x"               default="-0.1"  />
+    <xacro:arg name="gps_y"               default="0.05"  />
+    <xacro:arg name="gps_z"               default="0.07"  />
+    <xacro:arg name="gps_roll"            default="0"     />
+    <xacro:arg name="gps_pitch"           default="0"     />
+    <xacro:arg name="gps_yaw"             default="0"     />
+    <xacro:property name="gps_pose" default="$(arg gps_x) $(arg gps_y) $(arg gps_z)" />
+    <xacro:property name="gps_orientation" default="$(arg gps_roll) $(arg gps_pitch) $(arg gps_yaw)" />
     <!-- SCOUT mini wheel 3D file -->
     <xacro:include filename="$(find scout_description)/urdf/scout_mini_wheel_1.xacro" />
@@ -155,13 +175,13 @@
     <!-- SENSORS -->
     <!-- 2D hokuyo lidar -->
-    <xacro:if value="$(arg 2d_lidar)" >
+    <xacro:if value="$(arg hokuyo_lidar)" >
         <xacro:include filename="$(find scout_description)/urdf/hokuyo_2d.xacro" />
-        <xacro:hokuyo_lidar parent_link="base_link" topicName="$(arg 2d_lidar_topic)" visualize="$(arg visualize)" gpu="${gpu}">
+        <xacro:hokuyo_lidar parent_link="base_link" visualize="$(arg visualize)" gpu="${gpu}">
             <origin xyz="${lidar_pose}" rpy="${lidar_orientation}" />
         </xacro:hokuyo_lidar>
     </xacro:if>
     <!-- 3D Velodyne lidar -->
-    <xacro:if value="$(arg 3d_lidar)" >
-        <xacro:include filename="$(find scout_description)/urdf/$(arg 3d_lidar_name).xacro" />
+    <xacro:if value="$(arg velodyne_lidar)" >
+        <xacro:include filename="$(find scout_description)/urdf/$(arg velodyne_lidar_name).xacro" />
         <xacro:scout_3d_lidar parent_link="base_link" visualize="$(arg visualize)" gpu="${gpu}" xyz="${lidar_pose}" rpy="${lidar_orientation}" />
     </xacro:if>
@@ -169,11 +189,11 @@
     <xacro:if value="$(arg camera)" >
         <xacro:include filename="$(find scout_description)/urdf/$(arg camera_name).xacro" />
-        <xacro:scout_camera parent_link="base_link" name="camera" topics_ns="camera" publish_pointcloud="$(arg camera_pointcloud)" visualize="$(arg visualize)" xyz="$(arg camera_pose)" rpy="$(arg camera_orientation)" />
+        <xacro:scout_camera parent_link="base_link" name="camera" topics_ns="camera" publish_pointcloud="$(arg camera_pointcloud)" visualize="$(arg visualize)" xyz="${camera_pose}" rpy="${camera_orientation}" />
     </xacro:if>
     <!-- IMU -->
     <xacro:if value="$(arg imu)" >
         <xacro:include filename="$(find scout_description)/urdf/imu.xacro" />
-        <xacro:IMU parent_link="base_link" topicName="$(arg imu_topic)">
-            <origin xyz="$(arg imu_pose)" rpy="$(arg imu_orientation)" />
+        <xacro:IMU parent_link="base_link" >
+            <origin xyz="${imu_pose}" rpy="${imu_orientation}" />
         </xacro:IMU>
     </xacro:if>
@@ -181,6 +201,6 @@
     <xacro:if value="$(arg gps)" >
         <xacro:include filename="$(find scout_description)/urdf/gps.xacro" />
-        <xacro:GPS parent_link="base_link" topicName="$(arg gps_topic)">
-            <origin xyz="$(arg gps_pose)" rpy="$(arg gps_orientation)" />
+        <xacro:GPS parent_link="base_link" >
+            <origin xyz="${gps_pose}" rpy="${gps_orientation}" />
         </xacro:GPS>
     </xacro:if>
